File: leeco_lfaa/leeco_lfaa.kicad_pcb (KiCad board)
At the start: 2 copper layers, 0 parts

Commit message: Finished leeco_lfaa v1.0.
Parts:
- added MH1: MOUNTING_HOLE, leeco_lfaa:MOUNTING_HOLE, F.Cu at (91.4, 63.5)
- added MH2: MOUNTING_HOLE, leeco_lfaa:MOUNTING_HOLE, F.Cu at (182.9, 63.5)
- added MH3: MOUNTING_HOLE, leeco_lfaa:MOUNTING_HOLE, F.Cu at (91.4, 104.1)
- added MH4: MOUNTING_HOLE, leeco_lfaa:MOUNTING_HOLE, F.Cu at (182.9, 104.1)
- added P1: HEADER_02X04, leeco_lfaa:HEADER_02x04, F.Cu at (180.3, 83.8)
- added S1: LEECO_LFAA, leeco_lfaa:LEECO_LFAA, F.Cu at (167.6, 76.2)
- added S2: LEECO_LFAA, leeco_lfaa:LEECO_LFAA, F.Cu at (147.3, 76.2)
- added S3: LEECO_LFAA, leeco_lfaa:LEECO_LFAA, F.Cu at (127.0, 76.2)
- added S4: LEECO_LFAA, leeco_lfaa:LEECO_LFAA, F.Cu at (106.7, 76.2)
Routing:
- net VAA: track 0.00 -> 92.2 mm
- net /OUT3: track 0.00 -> 77.1 mm
- net /OUT2: track 0.00 -> 62.5 mm
- net /OUT1: track 0.00 -> 40.3 mm
- net /OUT0: track 0.00 -> 12.6 mm
- added copper zone on B.Cu, net VAA
- added copper zone on F.Cu, net VAA
Other:
- board outline added: 96.5 x 45.7 mm
- net class POWER added: clearance 0.254, trace_width 0.8128, via_dia 0.889, via_drill 0.635
- board text added: "Janelia Valve Board leeco_lfaa 09/2015 version 1.0"
- board text added: "VALVE 0"
- board text added: "VALVE 1"
- board text added: "VALVE 2"
- board text added: "VALVE 3"
- board text added: "https://github.com/janelia-idf/valve_boards"
