File: leeco_lfaa/leeco_lfaa.sch (KiCad schematic (older format))
At the start: 0 parts

Commit message: Finished leeco_lfaa v1.0.
Parts:
- added MH1, MH2, MH3, MH4: MOUNTING_HOLE, leeco_lfaa:MOUNTING_HOLE, symbol MOUNTING_HOLE
- added P1: HEADER_02X04, leeco_lfaa:HEADER_02x04, symbol HEADER_02X04
- added S1, S2, S3, S4: LEECO_LFAA, leeco_lfaa:LEECO_LFAA, symbol LEECO_LFAA
Connections:
- net labels added: OUT0, OUT1, OUT2, OUT3, VAA
- wire segments 0 -> 19
- no-connect marks 0 -> 4
Changed lines of the file:
@@
 LIBS:contrib
 LIBS:valves
+LIBS:components
+LIBS:leeco_lfaa
+LIBS:leeco_lfaa-cache
 EELAYER 25 0
 EELAYER END
@@
 Comment4 ""
 $EndDescr
+$Comp
+L VAA #PWR2
+U 1 1 55F1C05C
+P 3500 2700
+F 0 "#PWR2" H 3500 2550 50  0001 C CNN
+F 1 "VAA" H 3500 2850 50  0000 C CNN
+F 2 "" H 3500 2700 60  0000 C CNN
+F 3 "" H 3500 2700 60  0000 C CNN
+	1    3500 2700
+	1    0    0    -1
+$EndComp
+Wire Wire Line
+	3500 2700 3500 3100
+Wire Wire Line
+	3500 3100 3600 3100
+Wire Wire Line
+	3600 3000 3500 3000
+Connection ~ 3500 3000
+Wire Wire Line
+	3600 2900 3500 2900
+Connection ~ 3500 2900
+Wire Wire Line
+	3600 2800 3500 2800
+Connection ~ 3500 2800
+$Comp
+L VAA #PWR1
+U 1 1 55F1C0B2
+P 5050 2050
+F 0 "#PWR1" H 5050 1900 50  0001 C CNN
+F 1 "VAA" H 5050 2200 50  0000 C CNN
+F 2 "" H 5050 2050 60  0000 C CNN
+F 3 "" H 5050 2050 60  0000 C CNN
+	1    5050 2050
+	1    0    0    -1
+$EndComp
+Wire Wire Line
+	5150 3650 5050 3650
+Wire Wire Line
+	5050 3650 5050 2050
+Wire Wire Line
+	5150 3150 5050 3150
+Connection ~ 5050 3150
+Wire Wire Line
+	5150 2650 5050 2650
+Connection ~ 5050 2650
+Wire Wire Line
+	5150 2150 5050 2150
+Connection ~ 5050 2150
+Wire Wire Line
+	5150 2250 4800 2250
+Wire Wire Line
+	4100 2800 4200 2800
+Wire Wire Line
+	4100 2900 4200 2900
+Wire Wire Line
+	4100 3000 4200 3000
+Wire Wire Line
+	4100 3100 4200 3100
+Text Label 4200 2800 0    60   ~ 0
+OUT0
+Text Label 4200 2900 0    60   ~ 0
+OUT1
+Text Label 4200 3000 0    60   ~ 0
+OUT2
+Text Label 4200 3100 0    60   ~ 0
+OUT3
+Text Label 4800 2250 0    60   ~ 0
+OUT0
+Wire Wire Line
+	5150 2750 4800 2750
+Wire Wire Line
+	5150 3250 4800 3250
+Wire Wire Line
+	5150 3750 4800 3750
+Text Label 4800 2750 0    60   ~ 0
+OUT1
+Text Label 4800 3250 0    60   ~ 0
+OUT2
+Text Label 4800 3750 0    60   ~ 0
+OUT3
+$Comp
+L PWR_FLAG #FLG1
+U 1 1 55F1C4E9
+P 3250 2850
+F 0 "#FLG1" H 3250 2945 50  0001 C CNN
+F 1 "PWR_FLAG" H 3250 3030 50  0000 C CNN
+F 2 "" H 3250 2850 60  0000 C CNN
+F 3 "" H 3250 2850 60  0000 C CNN
+	1    3250 2850
+	1    0    0    -1
+$EndComp
+Wire Wire Line
+	3500 2850 3250 2850
+Connection ~ 3500 2850
+$Comp
+L HEADER_02X04 P1
+U 1 1 55F1C857
+P 3850 2950
+F 0 "P1" H 3850 3200 50  0000 C CNN
+F 1 "HEADER_02X04" H 3850 2700 50  0000 C CNN
+F 2 "leeco_lfaa:HEADER_02x04" H 3850 1750 60  0001 C CNN
+F 3 "" H 3850 1750 60  0000 C CNN
+F 4 "digikey" H 3950 3300 60  0001 C CNN "Vendor"
+F 5 "732-5395-ND" H 4050 3400 60  0001 C CNN "PartNumber"
+F 6 "CONN HEADER 8POS 2.54" H 4150 3500 60  0001 C CNN "Description"
+	1    3850 2950
+	1    0    0    -1
+$EndComp
+$Comp
+L LEECO_LFAA S1
+U 1 1 55F1CBA0
+P 5350 2200
+F 0 "S1" H 5350 2350 50  0000 C CNN
+F 1 "LEECO_LFAA" V 5450 2200 50  0000 C CNN
+F 2 "leeco_lfaa:LEECO_LFAA" H 5250 2250 60  0001 C CNN
+F 3 "" H 5350 2350 60  0000 C CNN
+F 4 "digikey" H 5450 2450 60  0001 C CNN "Vendor"
+F 5 "ED1013-ND" H 5550 2550 60  0001 C CNN "PartNumber"
+F 6 "CONN RECEPT PIN .032-.046in .240in" H 5650 2650 60  0001 C CNN "Description"
+	1    5350 2200
+	1    0    0    -1
+$EndComp
+$Comp
+L LEECO_LFAA S2
+U 1 1 55F1CCA2
+P 5350 2700
+F 0 "S2" H 5350 2850 50  0000 C CNN
+F 1 "LEECO_LFAA" V 5450 2700 50  0000 C CNN
+F 2 "leeco_lfaa:LEECO_LFAA" H 5250 2750 60  0001 C CNN
+F 3 "" H 5350 2850 60  0000 C CNN
+F 4 "digikey" H 5450 2950 60  0001 C CNN "Vendor"
+F 5 "ED1013-ND" H 5550 3050 60  0001 C CNN "PartNumber"
+F 6 "CONN RECEPT PIN .032-.046in .240in" H 5650 3150 60  0001 C CNN "Description"
+	1    5350 2700
+	1    0    0    -1
+$EndComp
+$Comp
+L LEECO_LFAA S3
+U 1 1 55F1CCD5
+P 5350 3200
+F 0 "S3" H 5350 3350 50  0000 C CNN
+F 1 "LEECO_LFAA" V 5450 3200 50  0000 C CNN
+F 2 "leeco_lfaa:LEECO_LFAA" H 5250 3250 60  0001 C CNN
+F 3 "" H 5350 3350 60  0000 C CNN
+F 4 "digikey" H 5450 3450 60  0001 C CNN "Vendor"
+F 5 "ED1013-ND" H 5550 3550 60  0001 C CNN "PartNumber"
+F 6 "CONN RECEPT PIN .032-.046in .240in" H 5650 3650 60  0001 C CNN "Description"
+	1    5350 3200
+	1    0    0    -1
+$EndComp
+$Comp
+L LEECO_LFAA S4
+U 1 1 55F1CD07
+P 5350 3700
+F 0 "S4" H 5350 3850 50  0000 C CNN
+F 1 "LEECO_LFAA" V 5450 3700 50  0000 C CNN
+F 2 "leeco_lfaa:LEECO_LFAA" H 5250 3750 60  0001 C CNN
+F 3 "" H 5350 3850 60  0000 C CNN
+F 4 "digikey" H 5450 3950 60  0001 C CNN "Vendor"
+F 5 "ED1013-ND" H 5550 4050 60  0001 C CNN "PartNumber"
+F 6 "CONN RECEPT PIN .032-.046in .240in" H 5650 4150 60  0001 C CNN "Description"
+	1    5350 3700
+	1    0    0    -1
+$EndComp
+$Comp
+L MOUNTING_HOLE MH1
+U 1 1 55F1CE8D
+P 6100 2000
+F 0 "MH1" H 6100 2100 50  0000 C CNN
+F 1 "MOUNTING_HOLE" V 6200 2000 50  0000 C CNN
+F 2 "leeco_lfaa:MOUNTING_HOLE" H 6000 2000 60  0001 C CNN
+F 3 "" H 6100 2000 60  0000 C CNN
+	1    6100 2000
+	1    0    0    -1
+$EndComp
+$Comp
+L MOUNTING_HOLE MH2
+U 1 1 55F1CF04
+P 6100 2650
+F 0 "MH2" H 6100 2750 50  0000 C CNN
+F 1 "MOUNTING_HOLE" V 6200 2650 50  0000 C CNN
+F 2 "leeco_lfaa:MOUNTING_HOLE" H 6000 2650 60  0001 C CNN
+F 3 "" H 6100 2650 60  0000 C CNN
+	1    6100 2650
+	1    0    0    -1
+$EndComp
+$Comp
+L MOUNTING_HOLE MH3
+U 1 1 55F1CF74
+P 6100 3300
+F 0 "MH3" H 6100 3400 50  0000 C CNN
+F 1 "MOUNTING_HOLE" V 6200 3300 50  0000 C CNN
+F 2 "leeco_lfaa:MOUNTING_HOLE" H 6000 3300 60  0001 C CNN
+F 3 "" H 6100 3300 60  0000 C CNN
+	1    6100 3300
+	1    0    0    -1
+$EndComp
+$Comp
+L MOUNTING_HOLE MH4
+U 1 1 55F1CFC8
+P 6100 3950
+F 0 "MH4" H 6100 4050 50  0000 C CNN
+F 1 "MOUNTING_HOLE" V 6200 3950 50  0000 C CNN
+F 2 "leeco_lfaa:MOUNTING_HOLE" H 6000 3950 60  0001 C CNN
+F 3 "" H 6100 3950 60  0000 C CNN
+	1    6100 3950
+	1    0    0    -1
+$EndComp
+NoConn ~ 5900 2000
+NoConn ~ 5900 2650
+NoConn ~ 5900 3300
+NoConn ~ 5900 3950
 $EndSCHEMATC

Commit message: Updated to v4.
Parts:
- MH1, MH2, MH3, MH4: symbol MOUNTING_HOLE -> leeco_lfaa:MOUNTING_HOLE
- P1: symbol HEADER_02X04 -> leeco_lfaa:HEADER_02X04
- S1, S2, S3, S4: symbol LEECO_LFAA -> leeco_lfaa:LEECO_LFAA
Connections:
- wire segments 19 -> 26
Changed lines of the file:
@@
-EESchema Schematic File Version 2
-LIBS:power
-LIBS:device
-LIBS:transistors
-LIBS:conn
-LIBS:linear
-LIBS:regul
-LIBS:74xx
-LIBS:cmos4000
-LIBS:adc-dac
-LIBS:memory
-LIBS:xilinx
-LIBS:microcontrollers
-LIBS:dsp
-LIBS:microchip
-LIBS:analog_switches
-LIBS:motorola
-LIBS:texas
-LIBS:intel
-LIBS:audio
-LIBS:interface
-LIBS:digital-audio
-LIBS:philips
-LIBS:display
-LIBS:cypress
-LIBS:siliconi
-LIBS:opto
-LIBS:atmel
-LIBS:contrib
-LIBS:valves
-LIBS:components
-LIBS:leeco_lfaa
+EESchema Schematic File Version 4
 LIBS:leeco_lfaa-cache
-EELAYER 25 0
+EELAYER 26 0
 EELAYER END
 $Descr A 11000 8500
@@
 $EndDescr
 $Comp
-L VAA #PWR2
+L power:VAA #PWR2
 U 1 1 55F1C05C
 P 3500 2700
@@
 $EndComp
 Wire Wire Line
-	3500 2700 3500 3100
+	3500 2700 3500 2800
 Wire Wire Line
 	3500 3100 3600 3100
@@
 Connection ~ 3500 2800
 $Comp
-L VAA #PWR1
+L power:VAA #PWR1
 U 1 1 55F1C0B2
 P 5050 2050
@@
 	5150 3650 5050 3650
 Wire Wire Line
-	5050 3650 5050 2050
+	5050 3650 5050 3150
 Wire Wire Line
 	5150 3150 5050 3150
@@
 OUT3
 $Comp
-L PWR_FLAG #FLG1
+L power:PWR_FLAG #FLG1
 U 1 1 55F1C4E9
 P 3250 2850
@@
 Connection ~ 3500 2850
 $Comp
-L HEADER_02X04 P1
+L leeco_lfaa:HEADER_02X04 P1
 U 1 1 55F1C857
 P 3850 2950
@@
 $EndComp
 $Comp
-L LEECO_LFAA S1
+L leeco_lfaa:LEECO_LFAA S1
 U 1 1 55F1CBA0
 P 5350 2200
@@
 $EndComp
 $Comp
-L LEECO_LFAA S2
+L leeco_lfaa:LEECO_LFAA S2
 U 1 1 55F1CCA2
 P 5350 2700
@@
 $EndComp
 $Comp
-L LEECO_LFAA S3
+L leeco_lfaa:LEECO_LFAA S3
 U 1 1 55F1CCD5
 P 5350 3200
@@
 $EndComp
 $Comp
-L LEECO_LFAA S4
+L leeco_lfaa:LEECO_LFAA S4
 U 1 1 55F1CD07
 P 5350 3700
@@
 $EndComp
 $Comp
-L MOUNTING_HOLE MH1
+L leeco_lfaa:MOUNTING_HOLE MH1
 U 1 1 55F1CE8D
 P 6100 2000
@@
 $EndComp
 $Comp
-L MOUNTING_HOLE MH2
+L leeco_lfaa:MOUNTING_HOLE MH2
 U 1 1 55F1CF04
 P 6100 2650
@@
 $EndComp
 $Comp
-L MOUNTING_HOLE MH3
+L leeco_lfaa:MOUNTING_HOLE MH3
 U 1 1 55F1CF74
 P 6100 3300
@@
 $EndComp
 $Comp
-L MOUNTING_HOLE MH4
+L leeco_lfaa:MOUNTING_HOLE MH4
 U 1 1 55F1CFC8
 P 6100 3950
@@
 NoConn ~ 5900 3300
 NoConn ~ 5900 3950
+Wire Wire Line
+	3500 3000 3500 3100
+Wire Wire Line
+	3500 2900 3500 3000
+Wire Wire Line
+	3500 2800 3500 2850
+Wire Wire Line
+	5050 3150 5050 2650
+Wire Wire Line
+	5050 2650 5050 2150
+Wire Wire Line
+	5050 2150 5050 2050
+Wire Wire Line
+	3500 2850 3500 2900
 $EndSCHEMATC
